Commit message: Added inertia and beginnings of sensors... bro idk

File: ora_description/src/description/concept.urdf (robot description, URDF)
Before this commit: robot concept, 6 links, 5 joints
Links:
- added link imu_link; collision box size=0.1 0.1 0.1; visual box size=0.1 0.1 0.1
- link left_wheel: geometry collision cylinder length=${wheel_width} radius=${wheel_radius}; visual cylinder length=${wheel_width} radius=${wheel_radius}
- link right_wheel: geometry collision cylinder length=${wheel_width} radius=${wheel_radius}; visual cylinder length=${wheel_width} radius=${wheel_radius}
Joints:
- added joint imu_joint: type fixed, parent base_link, child imu_link, origin xyz=0 0 0.01
- joint left_wheel_joint: origin xyz=0 ${(box_width/2)+(wheel_length/2)} -0.05 rpy=${pi/2} 0 0 -> xyz=0 ${(box_width/2)+(wheel_width/2)} -0.05 rpy=${pi/2} 0 0
- joint right_wheel_joint: origin xyz=0 ${(-box_width/2)+(-wheel_length/2)} -0.05 rpy=${pi/2} 0 0 -> xyz=0 ${(-box_width/2)+(-wheel_width/2)} -0.05 rpy=${pi/2} 0 0

Commit message: the return of desc-testing

File: ora_description/src/description/concept.urdf (robot description, URDF)
Before this commit: robot concept, 7 links, 6 joints
Links:
- added link camera_depth_frame
- added link camera_link, mass 0.23; collision box size=0.015 0.130 0.022; visual box size=0.015 0.130 0.022
Joints:
- added joint camera_depth_joint: type fixed, parent camera_link, child camera_depth_frame, origin xyz=0 0 0 rpy=0 0 0
- added joint camera_joint: type fixed, parent base_link, child camera_link, origin xyz=${(box_length/2)-(0.015/2)} 0 ${(box_height/2)+(0.022/2)} rpy=0 0 0

Commit message: costmap beginnings

File: ora_description/src/description/concept.urdf (robot description, URDF)
Before this commit: robot concept, 9 links, 8 joints
Joints:
- joint left_wheel_joint: origin xyz=0 ${(box_width/2)+(wheel_width/2)} -0.05 rpy=${pi/2} 0 0 -> xyz=0 ${(box_width/2)+(wheel_width/2)} -0.051 rpy=${pi/2} 0 0
- joint right_wheel_joint: origin xyz=0 ${(-box_width/2)+(-wheel_width/2)} -0.05 rpy=${pi/2} 0 0 -> xyz=0 ${(-box_width/2)+(-wheel_width/2)} -0.051 rpy=${pi/2} 0 0

Commit message: add GPS sensor to URDF

File: ora_description/src/description/concept.urdf (robot description, URDF)
Before this commit: robot concept, 9 links, 8 joints
Links:
- added link gps_link; collision box size=0.1 0.1 0.1; visual box size=0.1 0.1 0.1
Joints:
- added joint gps_joint: type fixed, parent base_link, child gps_link, origin xyz=0 0 0.01

Commit message: finally starting to get somewhere?

File: ora_description/src/description/concept.urdf (robot description, URDF)
Before this commit: robot concept, 10 links, 9 joints
Joints:
- joint camera_depth_joint: origin xyz=0 0 0 rpy=0 0 0 -> xyz=0 0 0 rpy=${-pi/2} 0 ${-pi/2}

Commit message: bruh, the wheels were on backwards

File: ora_description/src/description/concept.urdf (robot description, URDF)
Before this commit: robot concept, 10 links, 9 joints
Joints:
- joint left_wheel_joint: origin xyz=0 ${(box_width/2)+(wheel_width/2)} -0.051 rpy=${pi/2} 0 0 -> xyz=0 ${(box_width/2)+(wheel_width/2)} -0.051 rpy=${-pi/2} 0 0
- joint right_wheel_joint: origin xyz=0 ${(-box_width/2)+(-wheel_width/2)} -0.051 rpy=${pi/2} 0 0 -> xyz=0 ${(-box_width/2)+(-wheel_width/2)} -0.051 rpy=${-pi/2} 0 0
