Commit message: update urdf to match real robot

File: ora_description/src/description/horizon.urdf (robot description, URDF)
Before this commit: robot horizon, 10 links, 9 joints
Links:
- added link sensor_tower; collision box size=${(1/12)/3.281} ${(1/12)/3.281} ${tower_length}; visual box size=${(1/12)/3.281} ${(1/12)/3.281} ${tower_length}
Joints:
- added joint sensor_tower_joint: type fixed, parent base_link, child sensor_tower, origin xyz=0 0 ${tower_length/2} rpy=0 0 0
- joint camera_joint: origin xyz=${(box_length/2)-(0.015/2)} 0 ${(box_height/2)+(0.022/2)} rpy=0 0 0 -> xyz=${((1/12)/3.281)} 0 ${(tower_length-((3/12)/3.281))+(0.022/2)} rpy=0 ${12*(pi/180)} 0
- joint front_caster_joint: origin xyz=0.3 0 -0.1 rpy=0 0 0 -> xyz=${(box_length/2)-((1/12)/3.281)} 0 ${-box_height/2} rpy=0 0 0
- joint gps_joint: origin xyz=0 0 0.01 -> xyz=0 0 ${tower_length}
- joint left_wheel_joint: origin xyz=0 ${(box_width/2)+(wheel_width/2)} -0.051 rpy=${-pi/2} 0 0 -> xyz=0 ${(box_width/2)+(wheel_width/2)} ${-(box_height/4)-0.001} rpy=${-pi/2} 0 0
- joint rear_caster_joint: origin xyz=-0.3 0 -0.1 rpy=0 0 0 -> xyz=${(-box_length/2)+((1/12)/3.281)} 0 ${-box_height/2} rpy=0 0 0
- joint right_wheel_joint: origin xyz=0 ${(-box_width/2)+(-wheel_width/2)} -0.051 rpy=${-pi/2} 0 0 -> xyz=0 ${(-box_width/2)+(-wheel_width/2)} ${-(box_height/4)-0.001} rpy=${-pi/2} 0 0
