Commit message: update dimensions in horizon_zed to match IRL

File: ora_description/src/description/horizon_zed.urdf (robot description, URDF)
Before this commit: robot horizon_zed, 9 links, 9 joints
Links:
- link front_caster: geometry collision sphere radius=${front_caster_radius}; visual sphere radius=${front_caster_radius}
- link rear_caster: geometry collision sphere radius=${rear_caster_radius}; visual sphere radius=${rear_caster_radius}
Joints:
- joint $(arg camera_name)_joint: origin xyz=${(1/12)/3.281} 0 ${(tower_length-((3/12)/3.281))+(0.022/2)} rpy=0 ${12*(pi/180)} 0 -> xyz=${(box_length/2)-((1/12)/3.281)} 0 ${tower_length+(0.022/2)} rpy=0 ${12*(pi/180)} 0
- joint front_caster_joint: origin xyz=${(box_length/2)-((1/12)/3.281)} 0 ${-box_height/2} rpy=0 0 0 -> xyz=${(box_length/2)-front_caster_radius} 0 ${-box_height/2} rpy=0 0 0
- joint gps_joint: origin xyz=0 0 ${tower_length} -> xyz=0 0 ${box_height/2}
- joint left_wheel_joint: origin xyz=0 ${(box_width/2)+(wheel_width/2)} ${-(box_height/4)-0.001} rpy=${-pi/2} 0 0 -> xyz=0 ${(box_width/2)+(wheel_width/2)} ${-(box_height/6)-0.001} rpy=${-pi/2} 0 0
- joint rear_caster_joint: origin xyz=${(-box_length/2)+((1/12)/3.281)} 0 ${-box_height/2} rpy=0 0 0 -> xyz=${(-box_length/2)+rear_caster_radius} 0 ${-box_height/2} rpy=0 0 0
- joint right_wheel_joint: origin xyz=0 ${(-box_width/2)+(-wheel_width/2)} ${-(box_height/4)-0.001} rpy=${-pi/2} 0 0 -> xyz=0 ${(-box_width/2)+(-wheel_width/2)} ${-(box_height/6)-0.001} rpy=${-pi/2} 0 0
- joint sensor_tower_joint: origin xyz=0 0 ${tower_length/2} rpy=0 0 0 -> xyz=${(box_length/2)-((1/12)/3.281)} 0 ${(tower_length/2)+(box_height/2)-((8/12)/3.281)} rpy=0 0 0

Commit message: made it look nicer (and didn't break anything, hopefully)

File: ora_description/src/description/horizon_zed.urdf (robot description, URDF)
Before this commit: robot horizon_zed, 9 links, 9 joints
Links:
- link sensor_tower: geometry collision box size=${(1 / 12) / 3.281} ${(1 / 12) / 3.281} ${tower_length}; visual box size=${(1 / 12) / 3.281} ${(1 / 12) / 3.281} ${tower_length}
Joints:
- joint $(arg camera_name)_joint: origin xyz=${(box_length/2)-((1/12)/3.281)} 0 ${tower_length+(0.022/2)} rpy=0 ${12*(pi/180)} 0 -> xyz=${(box_length / 2) - ((1 / 12) / 3.281)} 0 ${tower_length + (0.022 / 2)} rpy=0 ${12 * (pi / 180)} 0
- joint front_caster_joint: origin xyz=${(box_length/2)-front_caster_radius} 0 ${-box_height/2} rpy=0 0 0 -> xyz=${(box_length / 2) - front_caster_radius} 0 ${-box_height / 2} rpy=0 0 0
- joint gps_joint: origin xyz=0 0 ${box_height/2} -> xyz=0 0 ${box_height / 2}
- joint left_wheel_joint: origin xyz=0 ${(box_width/2)+(wheel_width/2)} ${-(box_height/6)-0.001} rpy=${-pi/2} 0 0 -> xyz=0 ${(box_width / 2) + (wheel_width / 2)} ${-(box_height / 6) - 0.001} rpy=${-pi / 2} 0 0
- joint rear_caster_joint: origin xyz=${(-box_length/2)+rear_caster_radius} 0 ${-box_height/2} rpy=0 0 0 -> xyz=${(-box_length / 2) + rear_caster_radius} 0 ${-box_height / 2} rpy=0 0 0
- joint right_wheel_joint: origin xyz=0 ${(-box_width/2)+(-wheel_width/2)} ${-(box_height/6)-0.001} rpy=${-pi/2} 0 0 -> xyz=0 ${(-box_width / 2) + (-wheel_width / 2)} ${-(box_height / 6) - 0.001} rpy=${-pi / 2} 0 0
- joint sensor_tower_joint: origin xyz=${(box_length/2)-((1/12)/3.281)} 0 ${(tower_length/2)+(box_height/2)-((8/12)/3.281)} rpy=0 0 0 -> xyz=${(box_length / 2) - ((1 / 12) / 3.281)} 0 ${(tower_length 2 ) + (box_height / 2) - ((8 / 12) / 3.281)} rpy=0 0 0

Commit message: update zed urdf

File: ora_description/src/description/horizon_zed.urdf (robot description, URDF)
Before this commit: robot horizon_zed, 9 links, 9 joints
Joints:
- joint $(arg camera_name)_joint: origin xyz=${(box_length / 2) - ((1 / 12) / 3.281)} 0 ${tower_length + (0.022 / 2)} rpy=0 ${12 * (pi / 180)} 0 -> xyz=${(-(14 / 12) / 3.281)} 0 ${((49 / 12) / 3.281)} rpy=0 ${40 * (pi / 180)} 0
- joint sensor_tower_joint: origin xyz=${(box_length / 2) - ((1 / 12) / 3.281)} 0 ${(tower_length 2 ) + (box_height / 2) - ((8 / 12) / 3.281)} rpy=0 0 0 -> xyz=${(box_length / 2) - ((1 / 12) / 3.281)} 0 ${(tower_length / 2) + (box_height / 2) - ((8 / 12) / 3.281)} rpy=0 0 0
